File: hardware/revI/flan36-right.kicad_pcb (KiCad board)
At the start: 2 copper layers, 113.4 x 91.3 mm, 46 parts, among them J1 JST_PH_S2B-PH-K-S, J2 nice!view, K01 CHOC v1, K02 CHOC v1, K03 CHOC v1, K04 CHOC v1, K05 CHOC v1, K11 CHOC v1, K12 CHOC v1, K13 CHOC v1, K14 CHOC v1, K15 CHOC v1, K21 CHOC v1, K22 CHOC v1, K23 CHOC v1, K24 CHOC v1, K25 CHOC v1, K30 CHOC v1, K31 CHOC v1, K32 CHOC v1, SW1 PCM12SMTR, SW2 TL3342, U1 nice!nano v2

Commit message: Install Campo back silkscreen on both revI boards
Add the R2 Campo pattern and the Flan36 plate to B.SilkS of both routed
boards as one "silkscreen-art" group, via a new installer that refuses
stale art or a second install and records validation/revI-silkscreen.json.
The routing check (pads, poses, outline, DRC/ERC/parity) passes and the
regenerated Gerber packages differ only in B_Silkscreen; copper, mask,
outline and drill data are unchanged apart from export dates. Proposal
generators now refuse boards that already carry installed art.

Co-Authored-By: Claude Opus 5.5 <noreply@anthropic.com>
Other:
- board text added: "EDUARDO RUIZ"
- board text added: "REV I · 2026"
- board text added: "RIGHT"

Commit message: Adopt the Flan logo, sign the boards and ship silkscreen editions
Build the Flan logo kit: the three-quarter tecla-flan mark beside
"flan" in Fraunces (OFL) outlined with HarfBuzz, in display and
silkscreen constructions. Install it on the back of both routed revI
boards as the flan-signature group with REV I, 2026, the half and
eduarbo.com, removing the Campo pattern. Routing, DRC/ERC/parity and
the base fabrication packages are re-verified.

Export six back-silkscreen editions (Asanoha, Kikko, Sayagata,
Seigaiha, Meandro, Vias) as separate Gerber packages, each composed
across both halves around the signature. Every edition and half passes
DRC with schematic parity, reads back exactly and differs from the
base package only in B_Silkscreen. Document editions, logo and credits.

Co-Authored-By: Claude Opus 5.5 <noreply@anthropic.com>
Other:
- board text added: "2026"
- board text added: "REV I"
- board text added: "eduarbo.com"
- board text removed: "EDUARDO RUIZ"
- board text removed: "REV I · 2026"

Commit message: Sign the boards by eduarbo and set the signature into each pattern
The back signature now credits "by", the eduarbo cube and "eduarbo" instead
of eduarbo.com. The cube comes from eduarbo.com's favicon; in one ink three
thin cuts keep its faces apart (tools/branding/eduarbo.py).

Editions no longer clear a rounded box around the signature. The pattern
stops along the signature's own outline (closed over 0.9 mm, 0.8 mm halo)
and calms down within 6 mm of it (Canvas.quiet): Vías dots shrink and are
never cut, Asanoha and Kikkō keep their jigumi and drop spokes, Meandro runs
straight, Seigaiha fans lose inner arcs and Sayagata its centre vias.
Without a quiet zone every pattern draws as before.

Boards, base and edition packages are regenerated: DRC, ERC and schematic
parity pass, and each edition still differs from the base only in
B_Silkscreen.

Co-Authored-By: Claude Opus 5.5 <noreply@anthropic.com>
Other:
- board text added: "by"
- board text added: "eduarbo"
- board text removed: "eduarbo.com"
