File: hardware/flan42/flan42-left.kicad_pcb (KiCad board)
At the start: 2 copper layers, 131.4 x 91.3 mm, 53 parts, among them J1 JST_PH_S2B-PH-K-S, J2 nice!view, K00 CHOC v1, K01 CHOC v1, K02 CHOC v1, K03 CHOC v1, K04 CHOC v1, K05 CHOC v1, K10 CHOC v1, K11 CHOC v1, K12 CHOC v1, K13 CHOC v1, K14 CHOC v1, K15 CHOC v1, K20 CHOC v1, K21 CHOC v1, K22 CHOC v1, K23 CHOC v1, K24 CHOC v1, K25 CHOC v1, K30 CHOC v1, K31 CHOC v1, K32 CHOC v1, SW1 PCM12SMTR, SW2 TL3342, U1 nice!nano v2

Commit message: Share revI libraries and models for Flan42 and rebuild it
The variant projects now point their library tables and footprint 3D
models at ${KIPRJMOD}/../revI/ instead of carrying copies, so
hardware/flan42/libraries and models are gone. Flan42 is rebuilt,
rerouted, signed, checked and exported with the current tools: KiCad
10.0.6 DRC, ERC and schematic parity stay at 0 violations and 0
unconnected items per half, the negative controls still reject their
mutations, and the Gerber/drill readback still matches 676 outline
segments and every hole. The router's link order follows DRC, so a few
added links differ slightly from the previous routing.

Tool changes for the family: the build receipt records each half's
routing and routed hash, which install_signature reads; smooth_routes
keeps pad centres, vias and existing track ends as chain breaks (a
merged chain could skip a through-hole pad); the grid router extends its
grid only for a variant outline beyond revI's (revI receipts regenerate
unchanged); the fastener rule now compares each edge point with the
Flan36 edge point it extends (Flan42 still gets H6).

Co-Authored-By: Claude Opus 5.5 <noreply@anthropic.com>
Routing:
- net /COL0: track 218.5 -> 213.8 mm
